File: Datalogger_Beehive/Version 2/Digital_Datalogger/Digital_Datalogger.kicad_sch (KiCad schematic)
At the start: 62 parts, among them U1 DS18B20, U10 DS18B20, U11 DS18B20, U12 DS18B20, U13 DS18B20, U14 DS18B20, U15 DS18B20, U16 DS18B20, U17 DS18B20, U18 DS18B20, U19 DS18B20, U2 DS18B20, U20 DS18B20, U21 DS18B20, U22 DS18B20, U23 DS18B20, U24 DS18B20, U25 DS18B20, U26 DS18B20, U27 DS18B20, U28 DS18B20, U29 DS18B20, U3 DS18B20, U30 DS18B20, U31 DS18B20, U32 DS18B20, U33 DS18B20, U34 DS18B20, U35 DS18B20, U36 DS18B20, U37 DS18B20, U38 DS18B20, U39 DS18B20, U4 DS18B20, U40 DS18B20, U41 DS18B20, U42 DS18B20, U43 DS18B20, U44 DS18B20, U45 DS18B20, U46 DS18B20, U47 DS18B20, U48 DS18B20, U49 DS18B20, U5 DS18B20, U50 DS18B20, U51 DS18B20, U52 DS18B20, U53 DS18B20, U54 DS18B20, U55 DS18B20, U56 DS18B20, U57 DS18B20, U58 DS18B20, U59 DS18B20, U6 DS18B20, U60 DS18B20, U7 DS18B20, U8 DS18B20, U9 DS18B20

Commit message: Tweaking
Parts:
- added A2: Adafruit_Feather_Generic, Module:Adafruit_Feather, symbol MCU_Module:Adafruit_Feather_Generic
- R1: footprint (none) -> Resistor_THT:R_Axial_DIN0614_L14.3mm_D5.7mm_P25.40mm_Horizontal
- U42, U50: footprint Package_TO_SOT_THT:TO-92_Inline -> 1_my_custom_symbol_library:DS18B20 Connector
Connections:
- net Earth: now also A1.16 (GND), A1.4 (GND), A2.4 (GND)
- net at R1.2, U1.1 (GND), U10.1 (GND)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: now also A1.2 (3V3), A2.2 (3V3)
- net at R1.1, U1.2 (DQ), U10.2 (DQ)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: now also A2.23 (D4)
- net at A1.10 (A5): now also A2.10 (A5)
- net at A1.11 (SCK/D24): now also A2.11 (SCK)
- net at A1.12 (MOSI/D23): now also A2.12 (MOSI)
- net at A1.13 (MISO/D22): now also A2.13 (MISO)
- net at A1.23 (D11): now also A2.25 (D6)
- net at A1.9 (A4): now also A2.9 (A4)
